File: Complex/PCB/game.kicad_pcb (KiCad board)
At the start: 2 copper layers, 20 parts, among them U1 ESP32_DevKit_30pin, U4 74HC595

Commit message: Add files via upload
Some minor changes
Other:
- board outline added: 64 x 55.5 mm
Changed lines of the file:
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@@
 		)
+	)
+	(gr_rect
+		(start 103 63)
+		(end 167 118.5)
+		(stroke
+			(width 0.05)
+			(type default)
+		)
+		(fill no)
+		(layer "Edge.Cuts")
 	)
 	(gr_text "${REFERENCE}"
